File: Hardware/main_board/main_board.kicad_sch (KiCad schematic)
At the start: 23 parts

Commit message: more main pcb work (changed pinout, added USB interface), additional reference docs
Parts:
- removed JP?: SolderJumper_2_Open, symbol Jumper:SolderJumper_2_Open
- added C? (x2): 100n, symbol Device:C
- added C?: 4.7u, symbol Device:C
- added C?: 10n, symbol Device:C
- added C? (x2): 47p, symbol Device:C
- added C? (x2): DNP, symbol Device:C
- added C?: 0.1u, symbol Device:C
- added FB?: FerriteBead, symbol Device:FerriteBead
- added J?: USB_A, symbol Connector:USB_A
- added J?: DEBUG, symbol Connector:Conn_01x05_Male
- added JP?: SolderJumper_2_Bridged, symbol Jumper:SolderJumper_2_Bridged
- added R? (x2): 1k, symbol Device:R_US
- added R? (x2): 27R, symbol Device:R_US
- added R?: 5k, symbol Device:R_US
- added SW?: SW_Push, symbol Switch:SW_Push
- added TP?: TestPoint, symbol Connector:TestPoint
- added U?: FT201XQ, Package_DFN_QFN:QFN-16-1EP_4x4mm_P0.65mm_EP2.1x2.1mm, symbol Interface_USB:FT201XQ
- added Y?: 32MHz, symbol Device:Crystal
- gave numbers to parts that had none: 22
Connections:
- net +3V3: now also J?.1 (Pin_1), JP?.2 (B), R?.1, R?.1
- net ALARM_ON: now also U1.9 (PA2); no longer U1.7 (PA0)
- net GND: now also C?.1, C?.1, C?.1, C?.1, C?.1, C?.1, C?.2, C?.2, C?.2, J?.4 (GND), J?.5 (Pin_5), J?.5 (Shield), SW?.1, U?.13 (GND), U?.17 (GND), U?.3 (GND)
- net GPS_RXD: now also U1.33 (PA10); no longer U1.36 (PA13)
- net RFID_DATA0: now also U1.6 (PB8); no longer U1.2 (PB4)
- net RFID_DATA1: now also U1.8 (PA1); no longer U1.3 (PB5)
- net RFID_NRST: now also U1.3 (PB5); no longer U1.1 (PB3)
- net RFID_TAG_IN_RANGE: now also U1.7 (PA0); no longer U1.4 (PB6)
- net at JP4.1 (A), U1.25 (VDDPA): now also JP?.1 (A)
- net NRST: now reaches C8.1, SW1.2, U1.18 (NRST)
- net NRST: now also J?.2 (Pin_2)
- net RCC_MASTERCLK_OUT: now reaches U1.16 (PA8)
- net RCC_MASTERCLK_OUT: now also TP?.1
- net at U1.26 (OSC_IN): now also C?.2, Y?.2
- net at U1.27 (OSC_OUT): now also C?.2, Y?.1
- net DEBUG_JTCK_SWCLK: now reaches U1.42 (PA14)
- net DEBUG_JTCK_SWCLK: now also J?.4 (Pin_4)
- net DEBUG_JTDI: now reaches U1.43 (PA15)
- net I2C1_SDA: now reaches U1.5 (PB7)
- net I2C1_SDA: now also R?.2, U?.2 (SDA)
- new net: C?.1, R?.2, SW?.2, U?.9 (~{RESET})
- new net: C?.2, C?.2, FB?.2, U?.10 (VCC)
- new net: C?.2, U?.1 (VCCIO), U?.8 (3V3OUT)
- new net: C?.1, J?.3 (D+), R?.1
- new net: R?.2, U?.6 (USBDP)
- new net: C?.1, J?.2 (D-), R?.1
- new net: R?.2, U?.7 (USBDM)
- new net DBUG_JTDO_SWO: U1.1 (PB3)
- new net DEBUG_JTMS_SWDIO: J?.3 (Pin_3), U1.36 (PA13)
- new net DEBUG_JTRST: U1.2 (PB4)
- new net I2C1_SCL: R?.2, U1.4 (PB6), U?.16 (SCL)
- new net USB_5V: C?.2, FB?.1, J?.1 (VBUS), R?.1
Other:
- note added: "MCU Decoupling Caps"
- note added: "NOTE: Base Station board only!"
- note added: "Subsystem Connectors"
- note added: "TO DO: -- RF stuff -- FTDI USB implementation"
- note added: "USB Interface"
- note removed: "TO DO: -- Select HSE/LSE -- RF stuff"
- moved on the sheet: J1, J2, J3
