File: Hardware/main_board/main_board.kicad_sch (KiCad schematic)
At the start: 47 parts, among them J1 ALARM, J2 RFID_CONN, J3 GPS_CONN, J4 USB_A, J5 DEBUG, SW1 SW_Push, SW2 SW_Push, U1 STM32WL55_UFQFPN48, U2 FT201XQ, Y1 32MHz

Commit message: split schematic into separate board
Parts:
- removed D1: LED, symbol Device:LED
- removed J2: RFID_CONN, symbol Connector:Conn_01x06_Male
- removed R1: 500R, symbol Device:R_US
- added C20: 47n, Capacitor_SMD:C_0603_1608Metric, symbol Device:C_Small
- added C21: 68p, Capacitor_SMD:C_0603_1608Metric, symbol Device:C_Small
- added C22: 0.7p, Capacitor_SMD:C_0805_2012Metric, symbol Device:C
- added C23: 2p, Capacitor_SMD:C_0805_2012Metric, symbol Device:C
- added C24: 68p, Capacitor_SMD:C_0805_2012Metric, symbol Device:C
- added C25: DNP, Capacitor_SMD:C_0805_2012Metric, symbol Device:C
- added C26, C27: 1000p, Capacitor_SMD:C_0805_2012Metric, symbol Device:C
- added C28: 4.7p, Capacitor_SMD:C_0805_2012Metric, symbol Device:C
- added C29: 3p, Capacitor_SMD:C_0805_2012Metric, symbol Device:C
- added C30: 5.1p, Capacitor_SMD:C_0805_2012Metric, symbol Device:C
- added C31: 1p, Capacitor_SMD:C_0805_2012Metric, symbol Device:C
- added C32: 56p, Capacitor_SMD:C_0805_2012Metric, symbol Device:C
- added C33, C34: 3.3p, Capacitor_SMD:C_0805_2012Metric, symbol Device:C
- added C38, C39, C40, C41, C42, C43: 1u, Capacitor_SMD:C_0805_2012Metric, symbol Device:C
- added C44, C45: 10u, Capacitor_SMD:C_1206_3216Metric, symbol Device:C
- added C46: 1u, Capacitor_SMD:C_0805_2012Metric, symbol Device:C_Small
- added C47: 1u, Capacitor_SMD:C_0603_1608Metric, symbol Device:C
- added D4: D, Diode_SMD:D_2010_5025Metric, symbol Device:D
- added D5, D6, D7, D8: LED, LED_SMD:LED_0805_2012Metric, symbol Device:LED
- added J2: RFID_CONN, Connector_PinHeader_2.54mm:PinHeader_2x04_P2.54mm_Vertical, symbol Connector:Conn_01x08_Male
- added J6: ANTENNA2, Connector_Coaxial:SMA_Amphenol_132289_EdgeMount, symbol Connector:Conn_Coaxial
- added J8: BATT, Connector_PinHeader_2.54mm:PinHeader_1x02_P2.54mm_Vertical, symbol Connector:Conn_01x02_Male
- added J9: RFShield_TwoPieces, Capacitor_SMD:C_0805_2012Metric, symbol Device:RFShield_TwoPieces
- added L2: 47n, Inductor_SMD:L_0805_2012Metric_Pad1.05x1.20mm_HandSolder, symbol Device:L
- added L3: 4.45n, Inductor_SMD:L_0805_2012Metric_Pad1.05x1.20mm_HandSolder, symbol Device:L
- added L4: 3.6n, Inductor_SMD:L_0805_2012Metric_Pad1.05x1.20mm_HandSolder, symbol Device:L
- added L5: 8.7n, Inductor_SMD:L_0805_2012Metric_Pad1.05x1.20mm_HandSolder, symbol Device:L
- added L6: 11n, Inductor_SMD:L_0805_2012Metric_Pad1.05x1.20mm_HandSolder, symbol Device:L
- added L7: 9.1n, Inductor_SMD:L_0805_2012Metric_Pad1.05x1.20mm_HandSolder, symbol Device:L
- added R12, R13, R14, R15: 200R, Resistor_SMD:R_0805_2012Metric_Pad1.20x1.40mm_HandSolder, symbol Device:R_Small_US
- added TP11, TP12, TP13, TP14, TP3, TP4, TP5, TP6, TP7: TestPoint, Connector_PinHeader_2.54mm:PinHeader_1x01_P2.54mm_Vertical, symbol Connector:TestPoint
- added U3: SKY13370-374LF, Package_DFN_QFN:DFN-6-1EP_2x2mm_P0.5mm_EP0.6x1.37mm, symbol new_symbols:SKY13370-374LF
- added U5: AP7370-50W5-7, new_footprints:SOT25, symbol new_symbols:AP7370-50W5-7
- added U6: S-1135A33-M5T1U, Package_TO_SOT_SMD:SOT-23-5_HandSoldering, symbol new_symbols:S-1135A33-M5T1U
- added U7, U8: AP22811BW5-7, new_footprints:SOT25, symbol new_symbols:AP22811BW5-7
- added U9: 74LVC1G04, Package_TO_SOT_SMD:SOT-23-5_HandSoldering, symbol 74xGxx:74LVC1G04
- C1, C19, C2: footprint (none) -> Capacitor_SMD:C_0603_1608Metric
- C10, C11, C12, C13, C14, C15, C16, C17, C18, C3, C4, C5, C6, C7, C8, C9: footprint (none) -> Capacitor_SMD:C_0805_2012Metric
- D2, FB1: footprint (none) -> LED_SMD:LED_0805_2012Metric
- J1: footprint (none) -> Connector_PinHeader_2.54mm:PinHeader_1x03_P2.54mm_Vertical
- J3: footprint (none) -> Connector_PinHeader_2.54mm:PinHeader_1x06_P2.54mm_Vertical
- J4: footprint (none) -> Connector_USB:USB_A_Molex_67643_Horizontal
- J5: footprint (none) -> Connector_PinHeader_2.54mm:PinHeader_1x05_P2.54mm_Vertical
- JP1, JP2, JP3, JP4, JP5: footprint (none) -> Jumper:SolderJumper-2_P1.3mm_Open_TrianglePad1.0x1.5mm
- L1: footprint (none) -> Inductor_SMD:L_0805_2012Metric_Pad1.05x1.20mm_HandSolder
- R2, R3, R4, R5, R6, R7: footprint (none) -> Resistor_SMD:R_0805_2012Metric_Pad1.20x1.40mm_HandSolder
- SW1, SW2: footprint (none) -> Connector_PinSocket_2.54mm:PinSocket_1x02_P2.54mm_Vertical
- TP1, TP2: footprint (none) -> Connector_PinHeader_2.54mm:PinHeader_1x01_P2.54mm_Vertical
- U1: footprint (none) -> Package_DFN_QFN:QFN-48-1EP_7x7mm_P0.5mm_EP5.6x5.6mm
- Y1: footprint (none) -> Oscillator:Oscillator_SMD_Abracon_ASE-4Pin_3.2x2.5mm
Connections:
- net +3V3: now also C41.1, C42.1, C46.1, R14.1, TP13.1, U6.5 (VOUT), U7.5 (IN), U9.5 (VCC)
- net +5V: now also C39.1, C40.1, C43.1, R15.2, TP14.1, U5.5 (VOUT), U6.1 (VIN), U6.3 (ON), U8.5 (IN); no longer J3.2 (Pin_2)
- net GND: now also C20.2, C21.2, C22.2, C25.2, C26.1, C27.2, C28.2, C30.2, C31.1, C33.2, C34.2, C38.2, C39.2, C40.2, C41.2, C42.2, C43.2, C44.2, C45.2, C46.2, C47.2, D5.1 (K), D6.1 (K), D7.1 (K), D8.1 (K), J2.7 (Pin_7), J2.8 (Pin_8), J6.2 (Ext), J8.2 (Pin_2), J9.1 (Shield), U3.5 (GND), U5.2 (GND), U5.3 (NC), U5.4 (NC), U6.2 (VSS), U6.4 (NC), U7.2 (GND), U8.2 (GND), U9.3 (GND)
- net GPS_STATE: now also J3.4 (Pin_4); no longer J3.6 (Pin_6)
- net GPS_TXD: now also J3.6 (Pin_6); no longer J3.4 (Pin_4)
- net RFID_DATA0: now also J2.3 (Pin_3)
- net RFID_DATA1: now also J2.4 (Pin_4)
- net RFID_NRST: now also J2.5 (Pin_5)
- net RFID_TAG_IN_RANGE: now also J2.6 (Pin_6)
- net at JP1.1 (A), JP4.1 (A), U1.25 (VDDPA): now also C47.1
- net RFSW_VC1: now reaches U1.10 (PA3)
- net RFSW_VC1: now also C26.2, TP11.1, U3.1 (VC1), U9.2
- net at U1.12 (PA4): now also TP3.1
- net GPS_~{PWR}: now reaches U1.13 (PA5)
- net GPS_~{PWR}: now also U8.4 (~{EN})
- net RFID_~{PWR}: now reaches U1.14 (PA6)
- net RFID_~{PWR}: now also U7.4 (~{EN})
- net at U1.15 (PA7): now also TP6.1
- net at U1.20 (RFI_P): now also C29.1, L6.2
- net at U1.21 (RFI_N): now also C28.1, L6.1
- net at U1.23 (RFO_HP): now also L3.1
- net at U1.24 (VR_PA): now also C20.1, C21.1, L2.1
- net at U1.38 (PC13): now also TP7.1
- net at U1.39 (PC14-OSC32_IN): now also TP5.1
- net at U1.40 (PC15-OSC32_OUT): now also TP4.1
- net RCC_MASTERCLK_OUT: no longer names the net of TP2.1, U1.16 (PA8)
- new net: C38.1, D4.1 (K), U5.1 (VIN)
- new net: D8.2 (A), R15.1
- new net: D7.2 (A), R14.2
- new net: C22.1, C23.1, L2.2, L3.2, L4.1
- new net: C23.2, C24.1, C30.1, L4.2
- new net: C24.2, L5.1
- new net: C25.1, L5.2, U3.4 (RF2)
- new net: D5.2 (A), R12.2
- new net: C32.2, C33.1, L7.1
- new net: C34.1, J6.1 (In), L7.2
- new net: C32.1, U3.2 (RFC)
- new net: C29.2, C31.2, U3.6 (RF1)
- new net: D4.2 (A), J8.1 (Pin_1)
- new net: D6.2 (A), R13.2
- new net +3V3_RFID: C44.1, J2.1 (Pin_1), R12.1, U7.1 (OUT)
- new net +5V_GPS: C45.1, J3.2 (Pin_2), R13.1, U8.1 (OUT)
- new net RFID_LED: J2.2 (Pin_2)
- new net RFSW_VC2: C27.1, TP12.1, U3.3 (VC2), U9.4
- no-connect marks 0 -> 2
Other:
- note added: "- This board assumes the high-power RF output configuration: this means the output pin is RFO_HP, and VR_PA is tied to VCC."
- note added: "50 Ω"
- note added: "BATT: 4 AA batteries in series to provide 2700 mAh at 6V."
- note added: "LEDs for debugging only; depopulate to conserve power on production device."
- note added: "MICROCONTROLLER STM32WL55CCU7 48-QFN EP"
- note added: "POWER"
- note added: "RF Design Notes:"
- note added: "SUBSYSTEM LOAD SWITCHES"
- note added: "These are just pin-header connections.. making connectors is hard"
- note added: "VC1=1 -> RF1 ON --> TX VC1=0 -> RF2 ON --> RX"
- note removed: "MCU: STM32WL55CCU7 48-QFN EP"
- note removed: "TO DO: -- RF stuff -- FTDI USB implementation"
- moved on the sheet: TP1, TP2
