File: Hardware/main_board/main_board_bodged.kicad_sch (KiCad schematic)
At the start: 116 parts, among them J1 ALARM, J2 RFID_CONN, J3 GPS_CONN, J4 USB_A, J5 DEBUG, J6 ANTENNA2, J7 Conn_01x04_Male, J8 BATT, SW1 SW_Push, SW2 SW_Push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

Commit message: safety commit
Parts:
- removed Y1: 32MHz, Oscillator:Oscillator_SMD_Abracon_ASE-4Pin_3.2x2.5mm, symbol Device:Crystal
- added Y1: Crystal_GND24, Oscillator:Oscillator_SMD_Abracon_ASE-4Pin_3.2x2.5mm, symbol Device:Crystal_GND24
- C17, C19: value DNP -> 22p
- gave numbers to parts that had none: 1
Connections:
- net GND: now also Y1.2, Y1.4
- net I2C1_SCL: now also J2.3 (Pin_3); no longer J7.1 (Pin_1)
- net RFID_DATA0: now also TP22.1, U1.35 (PA12); no longer J2.3 (Pin_3), U1.32 (PB12)
- net USART1_RX: now also J3.3 (Pin_3); no longer J3.6 (Pin_6)
- net USART1_TX: now also J7.1 (Pin_1); no longer J3.3 (Pin_3)
- net at C17.2, U1.27 (OSC_OUT): now also Y1.1
- net at C19.2, U1.26 (OSC_IN): now also Y1.3
Other:
- note added: "NOTE: Trace cut; Y1 pad 3 to C19, Y1 pad 1 to C17"
Changed lines of the file:
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@@
   (junction (at 24.13 261.62) (diameter 0) (color 0 0 0 0)
   )
+  (junction (at 90.17 153.67) (diameter 0) (color 0 0 0 0)
+  )
   (junction (at 57.15 44.45) (diameter 0) (color 0 0 0 0)
   )
@@
     (stroke (width 0) (type default) (color 0 0 0 0))
   )
-  (wire (pts (xy 87.63 48.26) (xy 87.63 55.88))
-    (stroke (width 0) (type default) (color 0 0 0 0))
-  )
   (polyline (pts (xy 20.32 274.32) (xy 20.32 276.86))
     (stroke (width 0) (type default) (color 0 0 0 0))
@@
     (stroke (width 0) (type default) (color 0 0 0 0))
   )
+  (wire (pts (xy 90.17 153.67) (xy 92.71 153.67))
+    (stroke (width 0) (type default) (color 0 0 0 0))
+  )
   (wire (pts (xy 191.77 85.09) (xy 191.77 90.17))
     (stroke (width 0) (type default) (color 0 0 0 0))
@@
     (stroke (width 0) (type default) (color 0 0 0 0))
   )
-  (wire (pts (xy 90.17 121.92) (xy 90.17 156.21))
+  (wire (pts (xy 90.17 121.92) (xy 90.17 153.67))
     (stroke (width 0) (type default) (color 0 0 0 0))
   )
@@
     (stroke (width 0) (type default) (color 0 0 0 0))
   )
+  (wire (pts (xy 90.17 153.67) (xy 90.17 156.21))
+    (stroke (width 0) (type default) (color 0 0 0 0))
+  )
   (wire (pts (xy 355.6 46.99) (xy 360.68 46.99))
     (stroke (width 0) (type default) (color 0 0 0 0))
@@
     (effects (font (size 2 2) bold italic) (justify left bottom))
   )
+  (text "NOTE: Trace cut; Y1 pad 3 to C19, Y1 pad 1 to C17\n"
+    (at 63.5 19.05 0)
+    (effects (font (size 1.27 1.27)) (justify left bottom))
+  )
   (text "RF Design Notes: " (at 175.26 59.69 0)
     (effects (font (size 1.27 1.27) italic) (justify left bottom))
@@
     )
   )
-  (global_label "RFID_DATA0" (shape input) (at 87.63 48.26 90) (fields_autoplaced)
-    (effects (font (size 1.27 1.27) (thickness 0.254) bold italic) (justify left))
-    (property "Intersheet References" "${INTERSHEET_REFS}" (id 0) (at 87.503 34.5757 90)
-      (effects (font (size 1.27 1.27) (thickness 0.254) bold italic) (justify left) hide)
-    )
-  )
   (global_label "RFID_~{PWR}" (shape input) (at 327.66 167.64 180) (fields_autoplaced)
     (effects (font (size 1.27 1.27)) (justify right))
@@
     )
   )
-  (global_label "USART1_TX" (shape input) (at 227.33 261.62 0) (fields_autoplaced)
+  (global_label "USART1_TX" (shape input) (at 175.26 217.17 0) (fields_autoplaced)
     (effects (font (size 1.27 1.27) (thickness 0.254) bold italic) (justify left))
-    (property "Intersheet References" "${INTERSHEET_REFS}" (id 0) (at 240.4096 261.493 0)
+    (property "Intersheet References" "${INTERSHEET_REFS}" (id 0) (at 188.3396 217.043 0)
       (effects (font (size 1.27 1.27) (thickness 0.254) bold italic) (justify left) hide)
     )
@@
     )
   )
-  (global_label "I2C1_SCL" (shape input) (at 175.26 217.17 0) (fields_autoplaced)
+  (global_label "I2C1_SCL" (shape input) (at 184.15 261.62 0) (fields_autoplaced)
     (effects (font (size 1.27 1.27)) (justify left))
-    (property "Intersheet References" "${INTERSHEET_REFS}" (id 0) (at 186.4421 217.0906 0)
+    (property "Intersheet References" "${INTERSHEET_REFS}" (id 0) (at 195.3321 261.5406 0)
       (effects (font (size 1.27 1.27)) (justify left) hide)
     )
@@
     )
   )
-  (global_label "RFID_DATA0" (shape input) (at 184.15 261.62 0) (fields_autoplaced)
+  (global_label "RFID_DATA0" (shape input) (at 92.71 153.67 0) (fields_autoplaced)
     (effects (font (size 1.27 1.27)) (justify left))
-    (property "Intersheet References" "${INTERSHEET_REFS}" (id 0) (at 197.3883 261.5406 0)
+    (property "Intersheet References" "${INTERSHEET_REFS}" (id 0) (at 105.9483 153.5906 0)
       (effects (font (size 1.27 1.27)) (justify left) hide)
     )
@@
     )
   )
-  (global_label "USART1_RX" (shape input) (at 227.33 269.24 0) (fields_autoplaced)
+  (global_label "USART1_RX" (shape input) (at 227.33 261.62 0) (fields_autoplaced)
     (effects (font (size 1.27 1.27) (thickness 0.254) bold italic) (justify left))
-    (property "Intersheet References" "${INTERSHEET_REFS}" (id 0) (at 240.7119 269.113 0)
+    (property "Intersheet References" "${INTERSHEET_REFS}" (id 0) (at 240.7119 261.493 0)
       (effects (font (size 1.27 1.27) (thickness 0.254) bold italic) (justify left) hide)
     )
@@
     (pin "2")
   )
-  (symbol (lib_id "Device:Crystal") (at 71.12 33.02 0) (unit 1)
-    (in_bom yes) (on_board yes) (fields_autoplaced)
-    (property "Reference" "Y1" (id 0) (at 71.12 26.4881 0))
-    (property "Value" "32MHz" (id 1) (at 71.12 29.2632 0))
-    (property "Footprint" "Oscillator:Oscillator_SMD_Abracon_ASE-4Pin_3.2x2.5mm" (id 2) (at 71.12 33.02 0)
-      (effects (font (size 1.27 1.27)) hide)
-    )
-    (property "Datasheet" "~" (id 3) (at 71.12 33.02 0)
-      (effects (font (size 1.27 1.27)) hide)
-    )
-    (pin "1")
-    (pin "2")
-  )
   (symbol (lib_id "power:GND") (at 265.43 271.78 0) (unit 1)
     (in_bom yes) (on_board yes) (fields_autoplaced)
@@
     (pin "2")
   )
+  (symbol (lib_id "Device:Crystal_GND24") (at 71.12 33.02 0) (unit 1)
+    (in_bom yes) (on_board yes)
+    (property "Reference" "Y1" (id 0) (at 74.93 34.29 0))
+    (property "Value" "Crystal_GND24" (id 1) (at 91.44 29.21 0))
+    (property "Footprint" "Oscillator:Oscillator_SMD_Abracon_ASE-4Pin_3.2x2.5mm" (id 2) (at 71.12 33.02 0)
+      (effects (font (size 1.27 1.27)) hide)
+    )
+    (property "Datasheet" "~" (id 3) (at 71.12 33.02 0)
+      (effects (font (size 1.27 1.27)) hide)
+    )
+    (pin "1")
+    (pin "2")
+    (pin "3")
+    (pin "4")
+  )
   (symbol (lib_id "power:GND") (at 21.59 111.76 0) (unit 1)
     (in_bom yes) (on_board yes) (fields_autoplaced)
@@
     (pin "2")
   )
+  (symbol (lib_id "power:GND") (at 71.12 27.94 180) (unit 1)
+    (in_bom yes) (on_board yes) (fields_autoplaced)
+    (property "Reference" "#PWR0104" (id 0) (at 71.12 21.59 0)
+      (effects (font (size 1.27 1.27)) hide)
+    )
+    (property "Value" "GND" (id 1) (at 71.12 24.3355 0))
+    (property "Footprint" "" (id 2) (at 71.12 27.94 0)
+      (effects (font (size 1.27 1.27)) hide)
+    )
+    (property "Datasheet" "" (id 3) (at 71.12 27.94 0)
+      (effects (font (size 1.27 1.27)) hide)
+    )
+    (pin "1")
+  )
   (symbol (lib_id "Device:C") (at 41.91 184.15 0) (unit 1)
     (in_bom yes) (on_board yes) (fields_autoplaced)
@@
       (effects (font (size 1.27 1.27)) (justify left))
     )
-    (property "Value" "DNP" (id 1) (at 59.69 31.75 0)
+    (property "Value" "22p" (id 1) (at 59.69 31.75 0)
       (effects (font (size 1.27 1.27)) (justify left))
     )
@@
   (symbol (lib_id "Connector:TestPoint") (at 90.17 156.21 180) (unit 1)
     (in_bom yes) (on_board yes)
-    (property "Reference" "TP?" (id 0) (at 92.71 157.48 0))
+    (property "Reference" "TP22" (id 0) (at 92.71 157.48 0))
     (property "Value" "TestPoint" (id 1) (at 91.44 162.56 0)
       (effects (font (size 1.27 1.27)) hide)
@@
       (effects (font (size 1.27 1.27)) (justify left))
     )
-    (property "Value" "DNP" (id 1) (at 80.01 31.75 0)
+    (property "Value" "22p" (id 1) (at 80.01 31.75 0)
       (effects (font (size 1.27 1.27)) (justify left))
     )
@@
     (pin "2")
   )
+  (symbol (lib_id "power:GND") (at 71.12 38.1 0) (unit 1)
+    (in_bom yes) (on_board yes) (fields_autoplaced)
+    (property "Reference" "#PWR0105" (id 0) (at 71.12 44.45 0)
+      (effects (font (size 1.27 1.27)) hide)
+    )
+    (property "Value" "GND" (id 1) (at 71.12 42.6625 0))
+    (property "Footprint" "" (id 2) (at 71.12 38.1 0)
+      (effects (font (size 1.27 1.27)) hide)
+    )
+    (property "Datasheet" "" (id 3) (at 71.12 38.1 0)
+      (effects (font (size 1.27 1.27)) hide)
+    )
+    (pin "1")
+  )
   (symbol (lib_id "power:+3V3") (at 135.89 175.26 0) (unit 1)
     (in_bom yes) (on_board yes) (fields_autoplaced)
@@
       (reference "#PWR0103") (unit 1) (value "GND") (footprint "")
     )
+    (path "/756b0d12-883d-4a47-9773-55f69fbe3a37"
+      (reference "#PWR0104") (unit 1) (value "GND") (footprint "")
+    )
+    (path "/b2b68c35-a0ab-437f-8f8e-e7836fc67476"
+      (reference "#PWR0105") (unit 1) (value "GND") (footprint "")
+    )
     (path "/d74f20d8-b412-4a0b-82c3-52ca5cf3506c"
       (reference "C1") (unit 1) (value "4.7u") (footprint "Capacitor_SMD:C_0603_1608Metric")
@@
     )
     (path "/7d521a5c-eb08-45ad-ade4-d3734755183c"
-      (reference "C17") (unit 1) (value "DNP") (footprint "Capacitor_SMD:C_0603_1608Metric")
+      (reference "C17") (unit 1) (value "22p") (footprint "Capacitor_SMD:C_0603_1608Metric")
     )
     (path "/50b37ac3-c9f7-4d48-b534-94b77f2528c7"
@@
     )
     (path "/b19c8a34-f404-46c2-a83c-5315486ab0c9"
-      (reference "C19") (unit 1) (value "DNP") (footprint "Capacitor_SMD:C_0603_1608Metric")
+      (reference "C19") (unit 1) (value "22p") (footprint "Capacitor_SMD:C_0603_1608Metric")
     )
     (path "/2d9542ae-a09c-474b-a3c8-1c0507a1dcba"
@@
     )
     (path "/8398ae17-38b7-4311-9315-09c470c6af0f"
-      (reference "TP?") (unit 1) (value "TestPoint") (footprint "TestPoint:TestPoint_Pad_1.0x1.0mm")
+      (reference "TP22") (unit 1) (value "TestPoint") (footprint "TestPoint:TestPoint_Pad_1.0x1.0mm")
     )
     (path "/e3760479-0a57-413a-a85d-581fad0f8c75"
@@
       (reference "U8") (unit 1) (value "AP22811BW5-7") (footprint "new_footprints:SOT25")
     )
-    (path "/3f9ba76a-e880-4988-91ed-4af51b2b79d6"
-      (reference "Y1") (unit 1) (value "32MHz") (footprint "Oscillator:Oscillator_SMD_Abracon_ASE-4Pin_3.2x2.5mm")
+    (path "/651a6637-b8eb-400c-98e2-e30c05336858"
+      (reference "Y1") (unit 1) (value "Crystal_GND24") (footprint "Oscillator:Oscillator_SMD_Abracon_ASE-4Pin_3.2x2.5mm")
     )
   )
