File: Hardware/main_board/main_board_bodged.kicad_pcb (KiCad board)
At the start: 2 copper layers, 99.8 x 18.1 mm, 87 parts, among them J1 ALARM, J2 RFID_CONN, J3 GPS_CONN, J5 DEBUG, J6 ANTENNA2, J7 Conn_01x04_Male, J8 BATT, SW1 SW_Push, U1 STM32WL55_UFQFPN48, U3 SKY13370-374LF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

Commit message: safety commit
Parts:
- C17, C19: value DNP -> 22p
- Y1: value 32MHz -> Crystal_GND24
Connections:
- J3 pad 6: Net-(U1-Pad35) -> unconnected-(J3-Pad6)
- U1 pad 32: RFID_DATA0 -> unconnected-(U1-Pad32)
- U1 pad 35: Net-(U1-Pad35) -> RFID_DATA0
- Y1 pad 2: Net-(C19-Pad2) -> GND
- Y1 pad 3: (no net) -> Net-(C19-Pad2)
- Y1 pad 4: (no net) -> GND
Routing:
- net RFID_DATA0: track 0.00 -> 16.9 mm, vias 0 -> 1
- net Net-(U1-Pad35): track 16.9 -> 0.00 mm, vias 1 -> 0
- net Net-(C19-Pad2): track 6.78 -> 8.10 mm
- net GND: vias 80 -> 81
Changed lines of the file:
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@@
       (drillshape 0)
       (scaleselection 1)
-      (outputdirectory "mainboard_gerbers/")
+      (outputdirectory "main_bodge_gerber/")
     )
   )
@@
   (net 61 "USART1_TX")
   (net 62 "USART1_RX")
-  (net 63 "Net-(U1-Pad35)")
+  (net 63 "unconnected-(J3-Pad6)")
+  (net 64 "unconnected-(U1-Pad32)")
   (footprint "Inductor_SMD:L_0805_2012Metric_Pad1.05x1.20mm_HandSolder" (layer "F.Cu")
     (at 172.992 144.554 -90)
@@
       (effects (font (size 0.6 0.6) (thickness 0.15)))
     )
-    (fp_text value "DNP" (at 0 1.43 180) (layer "F.Fab")
+    (fp_text value "22p" (at 0 1.43 180) (layer "F.Fab")
       (effects (font (size 1 1) (thickness 0.15)))
     )
@@
       (net 13 "RFSW_VC2") (pinfunction "PB2") (pintype "unspecified"))
     (pad "32" smd roundrect locked (at 3.4375 -0.75 90) (size 0.875 0.25) (layers "F.Cu" "F.Paste" "F.Mask") (roundrect_rratio 0.25)
-      (net 31 "RFID_DATA0") (pinfunction "PB12") (pintype "unspecified"))
+      (net 64 "unconnected-(U1-Pad32)") (pinfunction "PB12") (pintype "unspecified"))
     (pad "33" smd roundrect locked (at 3.4375 -1.25 90) (size 0.875 0.25) (layers "F.Cu" "F.Paste" "F.Mask") (roundrect_rratio 0.25)
       (net 62 "USART1_RX") (pinfunction "PA10") (pintype "unspecified"))
@@
       (net 35 "GPS_STATE") (pinfunction "PA11") (pintype "unspecified"))
     (pad "35" smd roundrect locked (at 3.4375 -2.25 90) (size 0.875 0.25) (layers "F.Cu" "F.Paste" "F.Mask") (roundrect_rratio 0.25)
-      (net 63 "Net-(U1-Pad35)") (pinfunction "PA12") (pintype "unspecified"))
+      (net 31 "RFID_DATA0") (pinfunction "PA12") (pintype "unspecified"))
     (pad "36" smd roundrect locked (at 3.4375 -2.75 90) (size 0.875 0.25) (layers "F.Cu" "F.Paste" "F.Mask") (roundrect_rratio 0.25)
       (net 36 "DEBUG_JTMS_SWDIO") (pinfunction "PA13") (pintype "unspecified"))
@@
       (net 3 "GND") (pinfunction "Pin_5") (pintype "passive"))
     (pad "6" thru_hole oval locked (at 0 12.7 90) (size 1.7 1.7) (drill 1) (layers *.Cu *.Mask)
-      (net 63 "Net-(U1-Pad35)") (pinfunction "Pin_6") (pintype "passive"))
+      (net 63 "unconnected-(J3-Pad6)") (pinfunction "Pin_6") (pintype "passive"))
     (model "${KICAD6_3DMODEL_DIR}/Connector_PinHeader_2.54mm.3dshapes/PinHeader_1x06_P2.54mm_Vertical.wrl"
       (offset (xyz 0 0 0))
@@
       (effects (font (size 0.6 0.6) (thickness 0.15)))
     )
-    (fp_text value "DNP" (at 0 1.43) (layer "F.Fab")
+    (fp_text value "22p" (at 0 1.43) (layer "F.Fab")
       (effects (font (size 1 1) (thickness 0.15)))
     )
@@
       (effects (font (size 0.6 0.6) (thickness 0.15)))
     )
-    (fp_text value "32MHz" (at 0 2.45) (layer "F.Fab")
+    (fp_text value "Crystal_GND24" (at 0 2.45) (layer "F.Fab")
       (effects (font (size 1 1) (thickness 0.15)))
     )
@@
       (net 6 "Net-(C17-Pad2)") (pinfunction "1") (pintype "passive"))
     (pad "2" smd rect locked (at 1.05 0.825) (size 1.3 1.1) (layers "F.Cu" "F.Paste" "F.Mask")
-      (net 7 "Net-(C19-Pad2)") (pinfunction "2") (pintype "passive"))
-    (pad "3" smd rect locked (at 1.05 -0.825) (size 1.3 1.1) (layers "F.Cu" "F.Paste" "F.Mask"))
-    (pad "4" smd rect locked (at -1.05 -0.825) (size 1.3 1.1) (layers "F.Cu" "F.Paste" "F.Mask"))
+      (net 3 "GND") (pinfunction "2") (pintype "passive"))
+    (pad "3" smd rect locked (at 1.05 -0.825) (size 1.3 1.1) (layers "F.Cu" "F.Paste" "F.Mask")
+      (net 7 "Net-(C19-Pad2)") (pinfunction "3") (pintype "passive"))
+    (pad "4" smd rect locked (at -1.05 -0.825) (size 1.3 1.1) (layers "F.Cu" "F.Paste" "F.Mask")
+      (net 3 "GND") (pinfunction "4") (pintype "passive"))
     (model "${KICAD6_3DMODEL_DIR}/Oscillator.3dshapes/Oscillator_SMD_Abracon_ASE-4Pin_3.2x2.5mm.wrl"
       (offset (xyz 0 0 0))
@@
   (via (at 211.96 144.35) (size 0.8) (drill 0.4) (layers "F.Cu" "B.Cu") (free) (net 3))
   (via (at 166.175 137.2) (size 0.8) (drill 0.4) (layers "F.Cu" "B.Cu") (free) (net 3))
+  (via (at 184.57 133.29) (size 0.8) (drill 0.4) (layers "F.Cu" "B.Cu") (free) (net 3))
   (via (at 197.675 148.1) (size 0.8) (drill 0.4) (layers "F.Cu" "B.Cu") (free) (net 3))
   (via (at 205.2 138.1) (size 0.8) (drill 0.4) (layers "F.Cu" "B.Cu") (free) (net 3))
@@
   (segment (start 181.259039 137.790961) (end 181.259039 138.290961) (width 0.2) (layer "F.Cu") (net 6))
   (segment (start 181.259039 136.690961) (end 181.259039 137.790961) (width 0.2) (layer "F.Cu") (net 6))
-  (segment (start 184.674511 134.750489) (end 184.674511 135.375489) (width 0.2) (layer "F.Cu") (net 7))
-  (segment (start 183.725 136.325) (end 181.76 138.29) (width 0.2) (layer "F.Cu") (net 7))
+  (segment (start 182.67 135.58) (end 182.67 137.16) (width 0.25) (layer "F.Cu") (net 7))
+  (segment (start 181.71 137.99) (end 181.71 138.7525) (width 0.25) (layer "F.Cu") (net 7))
+  (segment (start 181.71 138.7525) (end 181.76 138.8025) (width 0.25) (layer "F.Cu") (net 7))
+  (segment (start 184.75 134.675) (end 185.75 133.675) (width 0.25) (layer "F.Cu") (net 7))
   (segment (start 181.76 138.29) (end 181.76 138.8025) (width 0.2) (layer "F.Cu") (net 7))
-  (segment (start 185.75 133.675) (end 184.674511 134.750489) (width 0.2) (layer "F.Cu") (net 7))
-  (segment (start 184.674511 135.375489) (end 183.725 136.325) (width 0.2) (layer "F.Cu") (net 7))
+  (segment (start 182.78 135.47) (end 182.67 135.58) (width 0.25) (layer "F.Cu") (net 7))
+  (segment (start 183.725 134.675) (end 184.75 134.675) (width 0.25) (layer "F.Cu") (net 7))
+  (segment (start 182.67 137.16) (end 181.84 137.99) (width 0.25) (layer "F.Cu") (net 7))
+  (segment (start 181.84 137.99) (end 181.71 137.99) (width 0.25) (layer "F.Cu") (net 7))
+  (segment (start 182.93 135.47) (end 182.78 135.47) (width 0.25) (layer "F.Cu") (net 7))
+  (segment (start 183.725 134.675) (end 182.93 135.47) (width 0.25) (layer "F.Cu") (net 7))
   (segment (start 185.777635 138.345) (end 187.507635 138.345) (width 0.8) (layer "F.Cu") (net 8))
   (segment (start 188.665 138.345) (end 189.23 137.78) (width 0.8) (layer "F.Cu") (net 8))
@@
   (segment (start 166.2504 147.77518) (end 166.425 147.60058) (width 0.2) (layer "B.Cu") (net 29))
   (segment (start 175.90048 149.00048) (end 180.725 149.00048) (width 0.2) (layer "B.Cu") (net 29))
+  (segment (start 176.404748 137.525489) (end 175.89 137.525489) (width 0.2) (layer "F.Cu") (net 31))
+  (segment (start 177.26 138.8025) (end 177.26 138.35) (width 0.2) (layer "F.Cu") (net 31))
+  (segment (start 175.49 137.38) (end 175.744511 137.38) (width 0.2) (layer "F.Cu") (net 31))
+  (segment (start 177.26 138.35) (end 176.45537 137.54537) (width 0.2) (layer "F.Cu") (net 31))
+  (segment (start 176.45537 137.54537) (end 176.424629 137.54537) (width 0.2) (layer "F.Cu") (net 31))
+  (segment (start 176.424629 137.54537) (end 176.404748 137.525489) (width 0.2) (layer "F.Cu") (net 31))
+  (segment (start 175.744511 137.38) (end 175.89 137.525489) (width 0.2) (layer "F.Cu") (net 31))
+  (via (at 175.49 137.38) (size 0.8) (drill 0.4) (layers "F.Cu" "B.Cu") (free) (net 31))
+  (segment (start 162.625 137.65) (end 163.86692 136.40808) (width 0.2) (layer "B.Cu") (net 31))
+  (segment (start 175.30808 136.40808) (end 175.49 136.59) (width 0.2) (layer "B.Cu") (net 31))
+  (segment (start 175.49 136.59) (end 175.49 137.38) (width 0.2) (layer "B.Cu") (net 31))
+  (segment (start 163.86692 136.40808) (end 175.30808 136.40808) (width 0.2) (layer "B.Cu") (net 31))
   (segment (start 180.18452 146.78548) (end 180.27 146.7) (width 0.2) (layer "F.Cu") (net 32))
   (segment (start 180.05 148.28) (end 180.225489 148.104511) (width 0.2) (layer "F.Cu") (net 32))
@@
   (segment (start 157.04596 135.60904) (end 155.005 137.65) (width 0.2) (layer "B.Cu") (net 62))
   (segment (start 176.298299 135.60904) (end 157.04596 135.60904) (width 0.2) (layer "B.Cu") (net 62))
-  (segment (start 176.404748 137.525489) (end 175.89 137.525489) (width 0.2) (layer "F.Cu") (net 63))
-  (segment (start 177.26 138.8025) (end 177.26 138.35) (width 0.2) (layer "F.Cu") (net 63))
-  (segment (start 175.49 137.38) (end 175.744511 137.38) (width 0.2) (layer "F.Cu") (net 63))
-  (segment (start 177.26 138.35) (end 176.45537 137.54537) (width 0.2) (layer "F.Cu") (net 63))
-  (segment (start 176.45537 137.54537) (end 176.424629 137.54537) (width 0.2) (layer "F.Cu") (net 63))
-  (segment (start 176.424629 137.54537) (end 176.404748 137.525489) (width 0.2) (layer "F.Cu") (net 63))
-  (segment (start 175.744511 137.38) (end 175.89 137.525489) (width 0.2) (layer "F.Cu") (net 63))
-  (via (at 175.49 137.38) (size 0.8) (drill 0.4) (layers "F.Cu" "B.Cu") (free) (net 63))
-  (segment (start 162.625 137.65) (end 163.86692 136.40808) (width 0.2) (layer "B.Cu") (net 63))
-  (segment (start 175.30808 136.40808) (end 175.49 136.59) (width 0.2) (layer "B.Cu") (net 63))
-  (segment (start 175.49 136.59) (end 175.49 137.38) (width 0.2) (layer "B.Cu") (net 63))
-  (segment (start 163.86692 136.40808) (end 175.30808 136.40808) (width 0.2) (layer "B.Cu") (net 63))
   (zone (net 41) (net_name "Net-(C25-Pad1)") (layer "F.Cu") (hatch edge 0.508)
     (priority 1)

Commit message: hahahhah
Connections:
- net ALARM_ON renamed LPUART1_NTX
- net GPS_STATE renamed PA11
- net I2C1_SCL renamed PB8
- net I2C1_SDA renamed PB7
- net RFID_DATA1 renamed PA1
- net RFID_LED renamed NC
- net RFID_NRST renamed PB5
- net RFID_TAG_IN_RANGE renamed PA0
- net RFSW_VC1 renamed LPUART1_NRX
- J3 pad 6: unconnected-(J3-Pad6) -> PA12
- U1 pad 35: RFID_DATA0 -> PA12
Routing:
- net RFID_DATA0: track 16.9 -> 0.00 mm, vias 1 -> 0
- net PA12: track 0.00 -> 16.9 mm, vias 0 -> 1
