File: Hardware/RFID_board/_autosave-RFID_board.kicad_sch (KiCad schematic)
At the start: 13 parts, among them J1 Conn_01x08_Male, Q1 2N3904, U1 ID-3LA

Commit message: finished rfid pcb
Connections:
- net +3V3: no longer R3.1
- net +3V3_RFID: now also R3.1
Changed lines of the file:
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@@
     (effects (font (size 2 2)) (justify left bottom))
+  )
+  (global_label "+3V3_RFID" (shape input) (at 160.02 60.96 90) (fields_autoplaced)
+    (effects (font (size 1.27 1.27)) (justify left))
+    (property "Intersheet References" "${INTERSHEET_REFS}" (id 0) (at 159.9406 48.2659 90)
+      (effects (font (size 1.27 1.27)) (justify left) hide)
+    )
   )
   (global_label "RFID_LED" (shape input) (at 96.52 60.96 0) (fields_autoplaced)
@@
       (effects (font (size 1.27 1.27)) (justify right) hide)
     )
-  )
-  (symbol (lib_id "power:+3V3") (at 160.02 60.96 0) (unit 1)
-    (in_bom yes) (on_board yes) (fields_autoplaced)
-    (property "Reference" "#PWR05" (id 0) (at 160.02 64.77 0)
-      (effects (font (size 1.27 1.27)) hide)
-    )
-    (property "Value" "+3V3" (id 1) (at 160.02 57.3555 0))
-    (property "Footprint" "" (id 2) (at 160.02 60.96 0)
-      (effects (font (size 1.27 1.27)) hide)
-    )
-    (property "Datasheet" "" (id 3) (at 160.02 60.96 0)
-      (effects (font (size 1.27 1.27)) hide)
-    )
-    (pin "1")
   )
   (symbol (lib_id "Device:R_Small_US") (at 182.88 64.77 90) (unit 1)
@@
       (reference "#PWR04") (unit 1) (value "GND") (footprint "")
     )
-    (path "/09bbea88-8bd7-48ec-baae-1b4a9a11a40e"
-      (reference "#PWR05") (unit 1) (value "+3V3") (footprint "")
-    )
     (path "/e86e4fae-9ca7-4857-a93c-bc6a3048f887"
