File: Hardware/alarm/alarm.kicad_sch (KiCad schematic)
At the start: 4 parts, among them Q1 Q_NMOS_DGS, Y1 Piezo Buzzer

Commit message: presentation
Parts:
- removed Q1: Q_NMOS_DGS, symbol Device:Q_NMOS_DGS
- removed R2: 1k, symbol Device:R_US
- removed Y1: Piezo Buzzer, symbol Device:Crystal
- added LS1: Speaker, symbol Device:Speaker
- added Q1: 2N3904, Package_TO_SOT_THT:TO-92_Inline, symbol Transistor_BJT:2N3904
- R1: value R_US -> 100R
Connections:
- net +3V3: now also LS1.1
- net GND: now also Q1.1 (E)
- net at R1.2: now also Q1.2 (B)
- net ALARM_CTRL renamed STM32_PWM
- new net: LS1.2, Q1.3 (C)
Changed lines of the file:
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@@
 (kicad_sch (version 20211123) (generator eeschema)
   (paper "A4")
-  (junction (at 151.13 72.39) (diameter 0) (color 0 0 0 0)
-  )
-  (junction (at 138.43 83.82) (diameter 0) (color 0 0 0 0)
-  )
-  (wire (pts (xy 138.43 72.39) (xy 151.13 72.39))
+  (wire (pts (xy 106.68 78.74) (xy 106.68 83.82))
     (stroke (width 0) (type default) (color 0 0 0 0))
   )
-  (wire (pts (xy 138.43 83.82) (xy 151.13 83.82))
+  (wire (pts (xy 77.47 88.9) (xy 91.44 88.9))
     (stroke (width 0) (type default) (color 0 0 0 0))
   )
-  (wire (pts (xy 110.49 92.71) (xy 123.19 92.71))
+  (wire (pts (xy 77.47 87.63) (xy 77.47 88.9))
     (stroke (width 0) (type default) (color 0 0 0 0))
   )
-  (wire (pts (xy 151.13 72.39) (xy 151.13 67.31))
+  (wire (pts (xy 106.68 72.39) (xy 106.68 76.2))
     (stroke (width 0) (type default) (color 0 0 0 0))
   )
-  (wire (pts (xy 110.49 91.44) (xy 110.49 92.71))
+  (wire (pts (xy 106.68 93.98) (xy 106.68 96.52))
     (stroke (width 0) (type default) (color 0 0 0 0))
   )
-  (wire (pts (xy 151.13 83.82) (xy 151.13 80.01))
-    (stroke (width 0) (type default) (color 0 0 0 0))
-  )
-  (wire (pts (xy 138.43 80.01) (xy 138.43 83.82))
-    (stroke (width 0) (type default) (color 0 0 0 0))
-  )
-  (wire (pts (xy 138.43 83.82) (xy 138.43 87.63))
-    (stroke (width 0) (type default) (color 0 0 0 0))
-  )
-  (wire (pts (xy 138.43 97.79) (xy 138.43 106.68))
-    (stroke (width 0) (type default) (color 0 0 0 0))
-  )
-  (label "ALARM_CTRL" (at 110.49 91.44 0)
+  (label "STM32_PWM" (at 77.47 87.63 0)
     (effects (font (size 1.27 1.27)) (justify left bottom))
   )
-  (symbol (lib_id "Device:Q_NMOS_DGS") (at 135.89 92.71 0) (unit 1)
+  (symbol (lib_id "Device:Speaker") (at 111.76 76.2 0) (unit 1)
     (in_bom yes) (on_board yes) (fields_autoplaced)
-    (property "Reference" "Q1" (id 0) (at 141.097 91.8015 0)
+    (property "Reference" "LS1" (id 0) (at 116.84 76.1999 0)
       (effects (font (size 1.27 1.27)) (justify left))
     )
-    (property "Value" "Q_NMOS_DGS" (id 1) (at 141.097 94.5766 0)
+    (property "Value" "Speaker" (id 1) (at 116.84 78.7399 0)
       (effects (font (size 1.27 1.27)) (justify left))
     )
-    (property "Footprint" "" (id 2) (at 140.97 90.17 0)
+    (property "Footprint" "" (id 2) (at 111.76 81.28 0)
       (effects (font (size 1.27 1.27)) hide)
     )
-    (property "Datasheet" "~" (id 3) (at 135.89 92.71 0)
+    (property "Datasheet" "~" (id 3) (at 111.506 77.47 0)
       (effects (font (size 1.27 1.27)) hide)
+    )
+    (pin "1")
+    (pin "2")
+  )
+  (symbol (lib_id "power:GND") (at 106.68 96.52 0) (unit 1)
+    (in_bom yes) (on_board yes) (fields_autoplaced)
+    (property "Reference" "#PWR02" (id 0) (at 106.68 102.87 0)
+      (effects (font (size 1.27 1.27)) hide)
+    )
+    (property "Value" "GND" (id 1) (at 106.68 101.6 0))
+    (property "Footprint" "" (id 2) (at 106.68 96.52 0)
+      (effects (font (size 1.27 1.27)) hide)
+    )
+    (property "Datasheet" "" (id 3) (at 106.68 96.52 0)
+      (effects (font (size 1.27 1.27)) hide)
+    )
+    (pin "1")
+  )
+  (symbol (lib_id "power:+3.3V") (at 106.68 72.39 0) (unit 1)
+    (in_bom yes) (on_board yes) (fields_autoplaced)
+    (property "Reference" "#PWR01" (id 0) (at 106.68 76.2 0)
+      (effects (font (size 1.27 1.27)) hide)
+    )
+    (property "Value" "+3.3V" (id 1) (at 106.68 67.31 0))
+    (property "Footprint" "" (id 2) (at 106.68 72.39 0)
+      (effects (font (size 1.27 1.27)) hide)
+    )
+    (property "Datasheet" "" (id 3) (at 106.68 72.39 0)
+      (effects (font (size 1.27 1.27)) hide)
+    )
+    (pin "1")
+  )
+  (symbol (lib_id "Device:R_US") (at 95.25 88.9 90) (unit 1)
+    (in_bom yes) (on_board yes) (fields_autoplaced)
+    (property "Reference" "R1" (id 0) (at 95.25 82.55 90))
+    (property "Value" "100R" (id 1) (at 95.25 85.09 90))
+    (property "Footprint" "" (id 2) (at 95.504 87.884 90)
+      (effects (font (size 1.27 1.27)) hide)
+    )
+    (property "Datasheet" "~" (id 3) (at 95.25 88.9 0)
+      (effects (font (size 1.27 1.27)) hide)
+    )
+    (pin "1")
+    (pin "2")
+  )
+  (symbol (lib_id "Transistor_BJT:2N3904") (at 104.14 88.9 0) (unit 1)
+    (in_bom yes) (on_board yes) (fields_autoplaced)
+    (property "Reference" "Q1" (id 0) (at 109.22 87.6299 0)
+      (effects (font (size 1.27 1.27)) (justify left))
+    )
+    (property "Value" "2N3904" (id 1) (at 109.22 90.1699 0)
+      (effects (font (size 1.27 1.27)) (justify left))
+    )
+    (property "Footprint" "Package_TO_SOT_THT:TO-92_Inline" (id 2) (at 109.22 90.805 0)
+      (effects (font (size 1.27 1.27) italic) (justify left) hide)
+    )
+    (property "Datasheet" "https://www.onsemi.com/pub/Collateral/2N3903-D.PDF" (id 3) (at 104.14 88.9 0)
+      (effects (font (size 1.27 1.27)) (justify left) hide)
     )
     (pin "1")
@@
     (pin "3")
   )
-  (symbol (lib_id "Device:Crystal") (at 151.13 76.2 90) (unit 1)
-    (in_bom yes) (on_board yes) (fields_autoplaced)
-    (property "Reference" "Y1" (id 0) (at 154.4574 75.2915 90)
-      (effects (font (size 1.27 1.27)) (justify right))
-    )
-    (property "Value" "Piezo Buzzer" (id 1) (at 154.4574 78.0666 90)
-      (effects (font (size 1.27 1.27)) (justify right))
-    )
-    (property "Footprint" "" (id 2) (at 151.13 76.2 0)
-      (effects (font (size 1.27 1.27)) hide)
-    )
-    (property "Datasheet" "~" (id 3) (at 151.13 76.2 0)
-      (effects (font (size 1.27 1.27)) hide)
-    )
-    (pin "1")
-    (pin "2")
-  )
-  (symbol (lib_id "power:+3V3") (at 151.13 67.31 0) (unit 1)
-    (in_bom yes) (on_board yes) (fields_autoplaced)
-    (property "Reference" "#PWR02" (id 0) (at 151.13 71.12 0)
-      (effects (font (size 1.27 1.27)) hide)
-    )
-    (property "Value" "+3V3" (id 1) (at 151.13 63.7055 0))
-    (property "Footprint" "" (id 2) (at 151.13 67.31 0)
-      (effects (font (size 1.27 1.27)) hide)
-    )
-    (property "Datasheet" "" (id 3) (at 151.13 67.31 0)
-      (effects (font (size 1.27 1.27)) hide)
-    )
-    (pin "1")
-  )
-  (symbol (lib_id "Device:R_US") (at 138.43 76.2 0) (unit 1)
-    (in_bom yes) (on_board yes) (fields_autoplaced)
-    (property "Reference" "R2" (id 0) (at 140.081 75.2915 0)
-      (effects (font (size 1.27 1.27)) (justify left))
-    )
-    (property "Value" "1k" (id 1) (at 140.081 78.0666 0)
-      (effects (font (size 1.27 1.27)) (justify left))
-    )
-    (property "Footprint" "" (id 2) (at 139.446 76.454 90)
-      (effects (font (size 1.27 1.27)) hide)
-    )
-    (property "Datasheet" "~" (id 3) (at 138.43 76.2 0)
-      (effects (font (size 1.27 1.27)) hide)
-    )
-    (pin "1")
-    (pin "2")
-  )
-  (symbol (lib_id "power:GND") (at 138.43 106.68 0) (unit 1)
-    (in_bom yes) (on_board yes) (fields_autoplaced)
-    (property "Reference" "#PWR01" (id 0) (at 138.43 113.03 0)
-      (effects (font (size 1.27 1.27)) hide)
-    )
-    (property "Value" "GND" (id 1) (at 138.43 111.2425 0))
-    (property "Footprint" "" (id 2) (at 138.43 106.68 0)
-      (effects (font (size 1.27 1.27)) hide)
-    )
-    (property "Datasheet" "" (id 3) (at 138.43 106.68 0)
-      (effects (font (size 1.27 1.27)) hide)
-    )
-    (pin "1")
-  )
-  (symbol (lib_id "Device:R_US") (at 127 92.71 90) (unit 1)
-    (in_bom yes) (on_board yes) (fields_autoplaced)
-    (property "Reference" "R1" (id 0) (at 127 87.8545 90))
-    (property "Value" "R_US" (id 1) (at 127 90.6296 90))
-    (property "Footprint" "" (id 2) (at 127.254 91.694 90)
-      (effects (font (size 1.27 1.27)) hide)
-    )
-    (property "Datasheet" "~" (id 3) (at 127 92.71 0)
-      (effects (font (size 1.27 1.27)) hide)
-    )
-    (pin "1")
-    (pin "2")
-  )
   (sheet_instances
     (path "/" (page "1"))
   )
   (symbol_instances
-    (path "/d712bda5-145f-4c1c-9a82-b42475fd77f3"
-      (reference "#PWR01") (unit 1) (value "GND") (footprint "")
+    (path "/4d9a5c15-b6c5-47a2-bb8c-738307f9e339"
+      (reference "#PWR01") (unit 1) (value "+3.3V") (footprint "")
     )
-    (path "/396b75b5-8301-434d-a10a-ad2aa7eccc47"
-      (reference "#PWR02") (unit 1) (value "+3V3") (footprint "")
+    (path "/1974c726-def2-42f6-bccb-1a0f7b6515d7"
+      (reference "#PWR02") (unit 1) (value "GND") (footprint "")
     )
-    (path "/00cf998a-a93b-44fd-a69a-31879d451d5c"
-      (reference "Q1") (unit 1) (value "Q_NMOS_DGS") (footprint "")
+    (path "/13fd50f6-1d47-4741-8619-6c6f05880696"
+      (reference "LS1") (unit 1) (value "Speaker") (footprint "")
     )
-    (path "/ff29d671-98a4-4862-895e-468b5261580f"
-      (reference "R1") (unit 1) (value "R_US") (footprint "")
+    (path "/900cb6c8-1d05-4537-a4f0-9a7cc1a2ea1c"
+      (reference "Q1") (unit 1) (value "2N3904") (footprint "Package_TO_SOT_THT:TO-92_Inline")
     )
-    (path "/46c31fef-8b6d-4892-b7d6-1b9818ed82f5"
-      (reference "R2") (unit 1) (value "1k") (footprint "")
-    )
-    (path "/24f7628d-681d-4f0e-8409-40a129e929d9"
-      (reference "Y1") (unit 1) (value "Piezo Buzzer") (footprint "")
+    (path "/4dee428b-9873-45f7-9e00-b3849b95bf1c"
+      (reference "R1") (unit 1) (value "100R") (footprint "")
     )
   )
